Commit message: Implement comprehensive AURA robot simulation package with ROS2 integration
Co-authored-by: sultanashaik6364 <sultanashaik6364@gmail.com>

File: urdf/aura_robot.urdf.xacro (robot description, xacro)
@@ -1,45 +1,190 @@
 <?xml version="1.0"?>
 <robot xmlns:xacro="http://www.ros.org/wiki/xacro" name="aura">
-  <xacro:property name="wheel_radius" value="0.03"/>
-  <xacro:property name="wheel_separation" value="0.2"/>
+  <!-- Include materials -->
+  <xacro:include filename="$(find aura_simulation)/urdf/materials.xacro" />
+  <!-- Robot dimensions -->
+  <xacro:property name="base_length" value="0.5"/>
+  <xacro:property name="base_width" value="0.5"/>
+  <xacro:property name="base_height" value="0.2"/>
+  <xacro:property name="wheel_radius" value="0.06"/>
+  <xacro:property name="wheel_width" value="0.04"/>
+  <xacro:property name="wheel_separation" value="0.4"/>
+  <xacro:property name="caster_radius" value="0.02"/>
+  <xacro:property name="lidar_height" value="0.05"/>
+  <xacro:property name="lidar_radius" value="0.06"/>
+  <xacro:property name="camera_size" value="0.03"/>
+  <!-- Base link - 0.5m x 0.5m x 0.2m box -->
   <link name="base_link">
     <visual>
-      <geometry><box size="0.3 0.2 0.1"/></geometry>
-      <material><color rgba="0.5 0.5 0.5 1.0"/></material>
-    </visual>
-    <collision>
-      <geometry><box size="0.3 0.2 0.1"/></geometry>
-    </collision>
-    <inertial>
-      <mass value="5.0"/>
-      <inertia ixx="0.1" iyy="0.1" izz="0.1" ixy="0.0" ixz="0.0" iyz="0.0"/>
-    </inertial>
-  </link>
-  <!-- lidar -->
+      <geometry>
+        <box size="${base_length} ${base_width} ${base_height}"/>
+      </geometry>
+      <material name="aura_blue"/>
+    </visual>
+    <collision>
+      <geometry>
+        <box size="${base_length} ${base_width} ${base_height}"/>
+      </geometry>
+    </collision>
+    <inertial>
+      <mass value="10.0"/>
+      <origin xyz="0 0 0" rpy="0 0 0"/>
+      <inertia ixx="0.208" ixy="0.0" ixz="0.0" iyy="0.208" iyz="0.0" izz="0.417"/>
+    </inertial>
+  </link>
+  <!-- Left drive wheel -->
+  <link name="left_wheel">
+    <visual>
+      <geometry>
+        <cylinder length="${wheel_width}" radius="${wheel_radius}"/>
+      </geometry>
+      <material name="wheel_black"/>
+    </visual>
+    <collision>
+      <geometry>
+        <cylinder length="${wheel_width}" radius="${wheel_radius}"/>
+      </geometry>
+    </collision>
+    <inertial>
+      <mass value="0.5"/>
+      <origin xyz="0 0 0" rpy="0 0 0"/>
+      <inertia ixx="0.0018" ixy="0.0" ixz="0.0" iyy="0.0018" iyz="0.0" izz="0.0036"/>
+    </inertial>
+  </link>
+  <!-- Right drive wheel -->
+  <link name="right_wheel">
+    <visual>
+      <geometry>
+        <cylinder length="${wheel_width}" radius="${wheel_radius}"/>
+      </geometry>
+      <material name="wheel_black"/>
+    </visual>
+    <collision>
+      <geometry>
+        <cylinder length="${wheel_width}" radius="${wheel_radius}"/>
+      </geometry>
+    </collision>
+    <inertial>
+      <mass value="0.5"/>
+      <origin xyz="0 0 0" rpy="0 0 0"/>
+      <inertia ixx="0.0018" ixy="0.0" ixz="0.0" iyy="0.0018" iyz="0.0" izz="0.0036"/>
+    </inertial>
+  </link>
+  <!-- Caster wheel -->
+  <link name="caster_wheel">
+    <visual>
+      <geometry>
+        <sphere radius="${caster_radius}"/>
+      </geometry>
+      <material name="caster_gray"/>
+    </visual>
+    <collision>
+      <geometry>
+        <sphere radius="${caster_radius}"/>
+      </geometry>
+    </collision>
+    <inertial>
+      <mass value="0.1"/>
+      <origin xyz="0 0 0" rpy="0 0 0"/>
+      <inertia ixx="0.00016" ixy="0.0" ixz="0.0" iyy="0.00016" iyz="0.0" izz="0.00016"/>
+    </inertial>
+  </link>
+  <!-- Lidar link (RPLiDAR A1 style) -->
   <link name="lidar_link">
-    <visual><geometry><cylinder length="0.05" radius="0.05"/></geometry></visual>
-  </link>
+    <visual>
+      <geometry>
+        <cylinder length="${lidar_height}" radius="${lidar_radius}"/>
+      </geometry>
+      <material name="lidar_red"/>
+    </visual>
+    <collision>
+      <geometry>
+        <cylinder length="${lidar_height}" radius="${lidar_radius}"/>
+      </geometry>
+    </collision>
+    <inertial>
+      <mass value="0.2"/>
+      <origin xyz="0 0 0" rpy="0 0 0"/>
+      <inertia ixx="0.00072" ixy="0.0" ixz="0.0" iyy="0.00072" iyz="0.0" izz="0.00144"/>
+    </inertial>
+  </link>
+  <!-- Camera link (placeholder) -->
+  <link name="camera_link">
+    <visual>
+      <geometry>
+        <box size="${camera_size} ${camera_size} ${camera_size}"/>
+      </geometry>
+      <material name="camera_gray"/>
+    </visual>
+    <collision>
+      <geometry>
+        <box size="${camera_size} ${camera_size} ${camera_size}"/>
+      </geometry>
+    </collision>
+    <inertial>
+      <mass value="0.1"/>
+      <origin xyz="0 0 0" rpy="0 0 0"/>
+      <inertia ixx="0.00015" ixy="0.0" ixz="0.0" iyy="0.00015" iyz="0.0" izz="0.00015"/>
+    </inertial>
+  </link>
+  <!-- Joints -->
+  <!-- Left wheel joint -->
+  <joint name="left_wheel_joint" type="continuous">
+    <parent link="base_link"/>
+    <child link="left_wheel"/>
+    <origin xyz="0 ${wheel_separation/2} -${base_height/2 + wheel_radius}" rpy="0 0 0"/>
+    <axis xyz="0 0 1"/>
+    <dynamics damping="0.1" friction="0.1"/>
+  </joint>
+  <!-- Right wheel joint -->
+  <joint name="right_wheel_joint" type="continuous">
+    <parent link="base_link"/>
+    <child link="right_wheel"/>
+    <origin xyz="0 -${wheel_separation/2} -${base_height/2 + wheel_radius}" rpy="0 0 0"/>
+    <axis xyz="0 0 1"/>
+    <dynamics damping="0.1" friction="0.1"/>
+  </joint>
+  <!-- Caster wheel joint -->
+  <joint name="caster_wheel_joint" type="fixed">
+    <parent link="base_link"/>
+    <child link="caster_wheel"/>
+    <origin xyz="${base_length/2 - 0.05} 0 -${base_height/2 + caster_radius}" rpy="0 0 0"/>
+  </joint>
+  <!-- Lidar joint -->
   <joint name="lidar_joint" type="fixed">
     <parent link="base_link"/>
     <child link="lidar_link"/>
-    <origin xyz="0 0 0.1"/>
-  </joint>
-  <!-- wheels -->
-  <link name="left_wheel"/>
-  <link name="right_wheel"/>
-  <joint name="left_wheel_joint" type="continuous">
-    <parent link="base_link"/>
-    <child link="left_wheel"/>
-    <origin xyz="0.0 0.1 0"/>
-    <axis xyz="0 1 0"/>
-  </joint>
-  <joint name="right_wheel_joint" type="continuous">
-    <parent link="base_link"/>
-    <child link="right_wheel"/>
-    <origin xyz="0.0 -0.1 0"/>
-    <axis xyz="0 1 0"/>
-  </joint>
-  <!-- Plugins -->
+    <origin xyz="0 0 ${base_height/2 + lidar_height/2}" rpy="0 0 0"/>
+  </joint>
+  <!-- Camera joint -->
+  <joint name="camera_joint" type="fixed">
+    <parent link="base_link"/>
+    <child link="camera_link"/>
+    <origin xyz="${base_length/2 + camera_size/2} 0 0" rpy="0 0 0"/>
+  </joint>
+  <!-- ROS2 Control transmissions -->
+  <transmission name="left_wheel_transmission">
+    <type>transmission_interface/SimpleTransmission</type>
+    <joint name="left_wheel_joint">
+      <hardwareInterface>hardware_interface/VelocityJointInterface</hardwareInterface>
+    </joint>
+    <actuator name="left_wheel_motor">
+      <hardwareInterface>hardware_interface/VelocityActuatorInterface</hardwareInterface>
+      <mechanicalReduction>1</mechanicalReduction>
+    </actuator>
+  </transmission>
+  <transmission name="right_wheel_transmission">
+    <type>transmission_interface/SimpleTransmission</type>
+    <joint name="right_wheel_joint">
+      <hardwareInterface>hardware_interface/VelocityJointInterface</hardwareInterface>
+    </joint>
+    <actuator name="right_wheel_motor">
+      <hardwareInterface>hardware_interface/VelocityActuatorInterface</hardwareInterface>
+      <mechanicalReduction>1</mechanicalReduction>
+    </actuator>
+  </transmission>
+  <!-- Gazebo plugins -->
   <gazebo>
+    <!-- Differential drive plugin -->
     <plugin name="diff_drive" filename="libgazebo_ros_diff_drive.so">
       <ros>
@@ -56,5 +201,10 @@
       <robot_base_frame>base_link</robot_base_frame>
       <publish_odom>true</publish_odom>
-    </plugin>
+      <publish_odom_tf>true</publish_odom_tf>
+      <publish_wheel_tf>false</publish_wheel_tf>
+      <odometry_source>world</odometry_source>
+      <ros2_control>true</ros2_control>
+    </plugin>
+    <!-- Lidar plugin -->
     <plugin name="lidar" filename="libgazebo_ros_ray_sensor.so">
       <ros>
@@ -68,11 +218,11 @@
             <samples>360</samples>
             <resolution>1</resolution>
-            <min_angle>-3.14</min_angle>
-            <max_angle>3.14</max_angle>
+            <min_angle>-3.14159</min_angle>
+            <max_angle>3.14159</max_angle>
           </horizontal>
         </scan>
         <range>
           <min>0.1</min>
-          <max>10.0</max>
+          <max>12.0</max>
           <resolution>0.01</resolution>
         </range>
@@ -83,4 +233,33 @@
         </noise>
       </ray>
+      <always_on>true</always_on>
+      <visualize>true</visualize>
+    </plugin>
+    <!-- Camera plugin -->
+    <plugin name="camera" filename="libgazebo_ros_camera.so">
+      <ros>
+        <namespace>/aura</namespace>
+        <remapping>image_raw:=camera/image_raw</remapping>
+        <remapping>camera_info:=camera/camera_info</remapping>
+      </ros>
+      <update_rate>30</update_rate>
+      <camera_name>aura_camera</camera_name>
+      <camera>camera_link</camera>
+      <always_on>true</always_on>
+      <visualize>true</visualize>
+      <image_width>640</image_width>
+      <image_height>480</image_height>
+      <image_format>R8G8B8</image_format>
+      <clip_near>0.1</clip_near>
+      <clip_far>100</clip_far>
+      <noise>
+        <type>gaussian</type>
+        <mean>0.0</mean>
+        <stddev>0.007</stddev>
+      </noise>
+    </plugin>
+    <!-- ROS2 Control plugin -->
+    <plugin name="ros2_control" filename="libgazebo_ros2_control.so">
+      <parameters>$(find aura_simulation)/config/aura_controllers.yaml</parameters>
     </plugin>
   </gazebo>

Commit message: Enhance AURA simulation package with detailed robot model and world
Co-authored-by: sultanashaik6364 <sultanashaik6364@gmail.com>

File: urdf/aura_robot.urdf.xacro (robot description, xacro)
@@ -1,46 +1,223 @@
 <?xml version="1.0"?>
 <robot xmlns:xacro="http://www.ros.org/wiki/xacro" name="aura">
-  <xacro:property name="wheel_radius" value="0.03"/>
-  <xacro:property name="wheel_separation" value="0.2"/>
+  <!-- Include materials -->
+  <xacro:include filename="$(find aura_simulation)/urdf/materials.xacro"/>
+  <!-- Robot properties -->
+  <xacro:property name="base_width" value="0.5"/>
+  <xacro:property name="base_length" value="0.5"/>
+  <xacro:property name="base_height" value="0.2"/>
+  <xacro:property name="base_mass" value="5.0"/>
+  <xacro:property name="wheel_radius" value="0.1"/>
+  <xacro:property name="wheel_width" value="0.04"/>
+  <xacro:property name="wheel_separation" value="0.4"/>
+  <xacro:property name="wheel_mass" value="1.0"/>
+  <xacro:property name="caster_radius" value="0.05"/>
+  <xacro:property name="caster_mass" value="0.5"/>
+  <xacro:property name="lidar_radius" value="0.05"/>
+  <xacro:property name="lidar_height" value="0.07"/>
+  <xacro:property name="lidar_mass" value="0.2"/>
+  <!-- Macro for wheel inertia -->
+  <xacro:macro name="cylinder_inertia" params="m r h">
+    <inertia ixx="${m*(3*r*r+h*h)/12}" ixy="0" ixz="0"
+             iyy="${m*(3*r*r+h*h)/12}" iyz="0"
+             izz="${m*r*r/2}"/>
+  </xacro:macro>
+  <!-- Macro for box inertia -->
+  <xacro:macro name="box_inertia" params="m x y z">
+    <inertia ixx="${m*(y*y+z*z)/12}" ixy="0" ixz="0"
+             iyy="${m*(x*x+z*z)/12}" iyz="0"
+             izz="${m*(x*x+y*y)/12}"/>
+  </xacro:macro>
+  <!-- Base Link -->
   <link name="base_link">
     <visual>
-      <geometry><box size="0.3 0.2 0.1"/></geometry>
-      <material><color rgba="0.5 0.5 0.5 1.0"/></material>
-    </visual>
-    <collision>
-      <geometry><box size="0.3 0.2 0.1"/></geometry>
-    </collision>
-    <inertial>
-      <mass value="5.0"/>
-      <inertia ixx="0.1" iyy="0.1" izz="0.1" ixy="0.0" ixz="0.0" iyz="0.0"/>
-    </inertial>
-  </link>
-  <!-- lidar -->
+      <origin xyz="0 0 ${base_height/2}" rpy="0 0 0"/>
+      <geometry>
+        <box size="${base_length} ${base_width} ${base_height}"/>
+      </geometry>
+      <material name="robot_base_color"/>
+    </visual>
+    <collision>
+      <origin xyz="0 0 ${base_height/2}" rpy="0 0 0"/>
+      <geometry>
+        <box size="${base_length} ${base_width} ${base_height}"/>
+      </geometry>
+    </collision>
+    <inertial>
+      <origin xyz="0 0 ${base_height/2}" rpy="0 0 0"/>
+      <mass value="${base_mass}"/>
+      <xacro:box_inertia m="${base_mass}" x="${base_length}" y="${base_width}" z="${base_height}"/>
+    </inertial>
+  </link>
+  <!-- Left Wheel -->
+  <link name="left_wheel">
+    <visual>
+      <origin xyz="0 0 0" rpy="${pi/2} 0 0"/>
+      <geometry>
+        <cylinder radius="${wheel_radius}" length="${wheel_width}"/>
+      </geometry>
+      <material name="wheel_color"/>
+    </visual>
+    <collision>
+      <origin xyz="0 0 0" rpy="${pi/2} 0 0"/>
+      <geometry>
+        <cylinder radius="${wheel_radius}" length="${wheel_width}"/>
+      </geometry>
+    </collision>
+    <inertial>
+      <origin xyz="0 0 0" rpy="${pi/2} 0 0"/>
+      <mass value="${wheel_mass}"/>
+      <xacro:cylinder_inertia m="${wheel_mass}" r="${wheel_radius}" h="${wheel_width}"/>
+    </inertial>
+  </link>
+  <!-- Right Wheel -->
+  <link name="right_wheel">
+    <visual>
+      <origin xyz="0 0 0" rpy="${pi/2} 0 0"/>
+      <geometry>
+        <cylinder radius="${wheel_radius}" length="${wheel_width}"/>
+      </geometry>
+      <material name="wheel_color"/>
+    </visual>
+    <collision>
+      <origin xyz="0 0 0" rpy="${pi/2} 0 0"/>
+      <geometry>
+        <cylinder radius="${wheel_radius}" length="${wheel_width}"/>
+      </geometry>
+    </collision>
+    <inertial>
+      <origin xyz="0 0 0" rpy="${pi/2} 0 0"/>
+      <mass value="${wheel_mass}"/>
+      <xacro:cylinder_inertia m="${wheel_mass}" r="${wheel_radius}" h="${wheel_width}"/>
+    </inertial>
+  </link>
+  <!-- Caster Wheel -->
+  <link name="caster_wheel">
+    <visual>
+      <origin xyz="0 0 0" rpy="0 0 0"/>
+      <geometry>
+        <sphere radius="${caster_radius}"/>
+      </geometry>
+      <material name="caster_color"/>
+    </visual>
+    <collision>
+      <origin xyz="0 0 0" rpy="0 0 0"/>
+      <geometry>
+        <sphere radius="${caster_radius}"/>
+      </geometry>
+    </collision>
+    <inertial>
+      <origin xyz="0 0 0" rpy="0 0 0"/>
+      <mass value="${caster_mass}"/>
+      <inertia ixx="${2*caster_mass*caster_radius*caster_radius/5}" ixy="0" ixz="0"
+               iyy="${2*caster_mass*caster_radius*caster_radius/5}" iyz="0"
+               izz="${2*caster_mass*caster_radius*caster_radius/5}"/>
+    </inertial>
+  </link>
+  <!-- Lidar Link -->
   <link name="lidar_link">
-    <visual><geometry><cylinder length="0.05" radius="0.05"/></geometry></visual>
-  </link>
+    <visual>
+      <origin xyz="0 0 0" rpy="0 0 0"/>
+      <geometry>
+        <cylinder radius="${lidar_radius}" length="${lidar_height}"/>
+      </geometry>
+      <material name="lidar_color"/>
+    </visual>
+    <collision>
+      <origin xyz="0 0 0" rpy="0 0 0"/>
+      <geometry>
+        <cylinder radius="${lidar_radius}" length="${lidar_height}"/>
+      </geometry>
+    </collision>
+    <inertial>
+      <origin xyz="0 0 0" rpy="0 0 0"/>
+      <mass value="${lidar_mass}"/>
+      <xacro:cylinder_inertia m="${lidar_mass}" r="${lidar_radius}" h="${lidar_height}"/>
+    </inertial>
+  </link>
+  <!-- Camera Link -->
+  <link name="camera_link">
+    <visual>
+      <origin xyz="0 0 0" rpy="0 0 0"/>
+      <geometry>
+        <box size="0.05 0.05 0.05"/>
+      </geometry>
+      <material name="camera_color"/>
+    </visual>
+    <collision>
+      <origin xyz="0 0 0" rpy="0 0 0"/>
+      <geometry>
+        <box size="0.05 0.05 0.05"/>
+      </geometry>
+    </collision>
+    <inertial>
+      <origin xyz="0 0 0" rpy="0 0 0"/>
+      <mass value="0.1"/>
+      <xacro:box_inertia m="0.1" x="0.05" y="0.05" z="0.05"/>
+    </inertial>
+  </link>
+  <!-- Joints -->
+  <!-- Left Wheel Joint -->
+  <joint name="left_wheel_joint" type="continuous">
+    <parent link="base_link"/>
+    <child link="left_wheel"/>
+    <origin xyz="0.0 ${wheel_separation/2} ${wheel_radius}" rpy="0 0 0"/>
+    <axis xyz="0 1 0"/>
+  </joint>
+  <!-- Right Wheel Joint -->
+  <joint name="right_wheel_joint" type="continuous">
+    <parent link="base_link"/>
+    <child link="right_wheel"/>
+    <origin xyz="0.0 ${-wheel_separation/2} ${wheel_radius}" rpy="0 0 0"/>
+    <axis xyz="0 1 0"/>
+  </joint>
+  <!-- Caster Wheel Joint -->
+  <joint name="caster_wheel_joint" type="fixed">
+    <parent link="base_link"/>
+    <child link="caster_wheel"/>
+    <origin xyz="${-base_length/2 + caster_radius} 0 ${caster_radius}" rpy="0 0 0"/>
+  </joint>
+  <!-- Lidar Joint -->
   <joint name="lidar_joint" type="fixed">
     <parent link="base_link"/>
     <child link="lidar_link"/>
-    <origin xyz="0 0 0.1"/>
-  </joint>
-  <!-- wheels -->
-  <link name="left_wheel"/>
-  <link name="right_wheel"/>
-  <joint name="left_wheel_joint" type="continuous">
-    <parent link="base_link"/>
-    <child link="left_wheel"/>
-    <origin xyz="0.0 0.1 0"/>
-    <axis xyz="0 1 0"/>
-  </joint>
-  <joint name="right_wheel_joint" type="continuous">
-    <parent link="base_link"/>
-    <child link="right_wheel"/>
-    <origin xyz="0.0 -0.1 0"/>
-    <axis xyz="0 1 0"/>
-  </joint>
-  <!-- Plugins -->
+    <origin xyz="0 0 ${base_height + lidar_height/2}" rpy="0 0 0"/>
+  </joint>
+  <!-- Camera Joint -->
+  <joint name="camera_joint" type="fixed">
+    <parent link="base_link"/>
+    <child link="camera_link"/>
+    <origin xyz="${base_length/2} 0 ${base_height/2}" rpy="0 0 0"/>
+  </joint>
+  <!-- Gazebo plugins and properties -->
+  <!-- Base link gazebo properties -->
+  <gazebo reference="base_link">
+    <material>Gazebo/Blue</material>
+  </gazebo>
+  <!-- Wheel gazebo properties -->
+  <gazebo reference="left_wheel">
+    <material>Gazebo/Black</material>
+    <mu1>0.8</mu1>
+    <mu2>0.8</mu2>
+  </gazebo>
+  <gazebo reference="right_wheel">
+    <material>Gazebo/Black</material>
+    <mu1>0.8</mu1>
+    <mu2>0.8</mu2>
+  </gazebo>
+  <gazebo reference="caster_wheel">
+    <material>Gazebo/Grey</material>
+    <mu1>0.1</mu1>
+    <mu2>0.1</mu2>
+  </gazebo>
+  <gazebo reference="lidar_link">
+    <material>Gazebo/Black</material>
+  </gazebo>
+  <gazebo reference="camera_link">
+    <material>Gazebo/Grey</material>
+  </gazebo>
+  <!-- Differential Drive Plugin -->
   <gazebo>
-    <plugin name="diff_drive" filename="libgazebo_ros_diff_drive.so">
+    <plugin name="differential_drive_controller" filename="libgazebo_ros_diff_drive.so">
       <ros>
         <namespace>/aura</namespace>
@@ -50,5 +227,7 @@
       <right_joint>right_wheel_joint</right_joint>
       <wheel_separation>${wheel_separation}</wheel_separation>
-      <wheel_radius>${wheel_radius}</wheel_radius>
+      <wheel_diameter>${2*wheel_radius}</wheel_diameter>
+      <max_wheel_torque>10</max_wheel_torque>
+      <max_wheel_acceleration>1.0</max_wheel_acceleration>
       <command_topic>cmd_vel</command_topic>
       <odometry_topic>odom</odometry_topic>
@@ -56,10 +235,13 @@
       <robot_base_frame>base_link</robot_base_frame>
       <publish_odom>true</publish_odom>
+      <publish_odom_tf>true</publish_odom_tf>
+      <publish_wheel_tf>false</publish_wheel_tf>
     </plugin>
-    <plugin name="lidar" filename="libgazebo_ros_ray_sensor.so">
-      <ros>
-        <namespace>/aura</namespace>
-        <remapping>scan:=scan</remapping>
-      </ros>
+  </gazebo>
+  <!-- Lidar Plugin -->
+  <gazebo reference="lidar_link">
+    <sensor type="ray" name="lidar_sensor">
+      <pose>0 0 0 0 0 0</pose>
+      <visualize>true</visualize>
       <update_rate>20</update_rate>
       <ray>
@@ -68,6 +250,6 @@
             <samples>360</samples>
             <resolution>1</resolution>
-            <min_angle>-3.14</min_angle>
-            <max_angle>3.14</max_angle>
+            <min_angle>-3.14159</min_angle>
+            <max_angle>3.14159</max_angle>
           </horizontal>
         </scan>
@@ -83,5 +265,41 @@
         </noise>
       </ray>
-    </plugin>
+      <plugin name="gazebo_ros_lidar_controller" filename="libgazebo_ros_ray_sensor.so">
+        <ros>
+          <namespace>/aura</namespace>
+          <remapping>~/out:=scan</remapping>
+        </ros>
+        <output_type>sensor_msgs/LaserScan</output_type>
+        <frame_name>lidar_link</frame_name>
+      </plugin>
+    </sensor>
+  </gazebo>
+  <!-- Camera Plugin -->
+  <gazebo reference="camera_link">
+    <sensor type="camera" name="camera_sensor">
+      <update_rate>30.0</update_rate>
+      <camera name="camera">
+        <horizontal_fov>1.3962634</horizontal_fov>
+        <image>
+          <width>800</width>
+          <height>600</height>
+          <format>R8G8B8</format>
+        </image>
+        <clip>
+          <near>0.02</near>
+          <far>300</far>
+        </clip>
+      </camera>
+      <plugin name="camera_controller" filename="libgazebo_ros_camera.so">
+        <ros>
+          <namespace>/aura</namespace>
+          <remapping>image_raw:=camera/image_raw</remapping>
+          <remapping>camera_info:=camera/camera_info</remapping>
+        </ros>
+        <camera_name>camera</camera_name>
+        <frame_name>camera_link</frame_name>
+        <hack_baseline>0.07</hack_baseline>
+      </plugin>
+    </sensor>
   </gazebo>
 </robot>
